File: FGINT-V3-MASTER-64/FGINT-V3-MASTER-64.kicad_pcb (KiCad board)
At the start: 2 copper layers, 139.7 x 128.3 mm, 48 parts, among them J1 OUT1-16, J10 ComGPIOB2, J11 OUT48-64, J12 ComGPIOA3, J13 ComGPIOB3, J14 9V - 12 DC, J15 Raspberry, J16 Exp 01, J17 Exp 02, J18 Exp 03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

Commit message: copyright @daweed added, routing modified
Routing:
- net GND: track 754.6 -> 774.2 mm, vias 0 -> 1
Other:
- rule pad_to_mask_clearance: 0.051 -> 0
- board text added: "rev. 1.1 - Master-64 - © Daweed Le Fermier produced: a320@movingminds.eu"

Commit message: Gerber-export files modified
Other:
- board text added: "rev. 3.1 - Master-64 - © Daweed Le Fermier pcb from: a320@movingminds.eu - 10/2021"
- board text removed: "rev. 1.1 - Master-64 - © Daweed Le Fermier produced: a320@movingminds.eu"
